Commit message: add cr3 bringup to mobile base

File: walkie2_ws/src/cr3_lowlevel_pkg/urdf/cr3_robot_w_gripper_for_walkie2.xacro (robot description, xacro)
@@ -37,7 +37,7 @@
     </visual>
     <collision>
-      <origin xyz="0 0 0" rpy="0 0 -1.57" />
-      <geometry>
-        <mesh filename="package://cr3_lowlevel_pkg/meshes/base_link.STL" />
+      <origin xyz="0 0.025 0.035" rpy="0 0 -1.57" />
+      <geometry>
+        <mesh filename="package://cr3_lowlevel_pkg/meshes/base_link_1.STL" scale="0.001 0.001 0.001"/>
       </geometry>
     </collision>
@@ -46,5 +46,5 @@
     <parent link="${parent_link}" />
     <child link="cr3_base_link" />
-    <origin xyz="0.20 0.0 0.0" rpy="0.0 0.0 3.14" />
+    <origin xyz="0.20 0.0 -0.3" rpy="0.0 0.0 3.14" />
   </joint>
   <link name="Link1">
@@ -171,5 +171,5 @@
       <origin xyz="0 0 0" rpy="0 0 0" />
       <geometry>
-        <mesh filename="package://cr3_lowlevel_pkg/meshes/Link5.STL" scale="1.1 1.3 1.3"/>
+        <mesh filename="package://cr3_lowlevel_pkg/meshes/Link5.STL" scale="1.1 1.1 1.1"/>
       </geometry>
     </collision>

File: walkie2_ws/src/walkie2_description/urdf/walkie2.xacro (robot description, xacro)
@@ -40,5 +40,5 @@
     <origin xyz="0.0 -0.194 -0.098" rpy="0 0 0"/>
     <geometry>
-      <mesh filename="package://walkie2_description/meshes/RM_1_1.stl" scale="0.001 0.001 0.001"/>
+      <mesh filename="package://walkie2_description/meshes/RM_1.stl" scale="0.001 0.001 0.001"/>
     </geometry>
     <material name="silver"/>
@@ -47,5 +47,5 @@
     <origin xyz="0.0 -0.194 -0.098" rpy="0 0 0"/>
     <geometry>
-      <mesh filename="package://walkie2_description/meshes/RM_1_1.stl" scale="0.001 0.001 0.001"/>
+      <mesh filename="package://walkie2_description/meshes/RM_1.stl" scale="0.001 0.001 0.001"/>
     </geometry>
   </collision>
@@ -60,5 +60,5 @@
     <origin xyz="0.0 0.194 -0.098" rpy="0 0 0"/>
     <geometry>
-      <mesh filename="package://walkie2_description/meshes/LM_1_1.stl" scale="0.001 0.001 0.001"/>
+      <mesh filename="package://walkie2_description/meshes/LM_1.stl" scale="0.001 0.001 0.001"/>
     </geometry>
     <material name="silver"/>
@@ -67,5 +67,5 @@
     <origin xyz="0.0 0.194 -0.098" rpy="0 0 0"/>
     <geometry>
-      <mesh filename="package://walkie2_description/meshes/LM_1_1.stl" scale="0.001 0.001 0.001"/>
+      <mesh filename="package://walkie2_description/meshes/LM_1.stl" scale="0.001 0.001 0.001"/>
     </geometry>
   </collision>
@@ -80,5 +80,5 @@
     <origin xyz="-0.197 0.0 -0.1955" rpy="0 0 0"/>
     <geometry>
-      <mesh filename="package://walkie2_description/meshes/lidar_1_1.stl" scale="0.001 0.001 0.001"/>
+      <mesh filename="package://walkie2_description/meshes/lidar_1.stl" scale="0.001 0.001 0.001"/>
     </geometry>
     <material name="silver"/>
@@ -87,5 +87,5 @@
     <origin xyz="-0.197 0.0 -0.1955" rpy="0 0 0"/>
     <geometry>
-      <mesh filename="package://walkie2_description/meshes/lidar_1_1.stl" scale="0.001 0.001 0.001"/>
+      <mesh filename="package://walkie2_description/meshes/lidar_1.stl" scale="0.001 0.001 0.001"/>
     </geometry>
   </collision>
@@ -100,5 +100,5 @@
     <origin xyz="0.016306 -0.0 -0.7855" rpy="0 0 0"/>
     <geometry>
-      <mesh filename="package://walkie2_description/meshes/CR3base_1_1.stl" scale="0.001 0.001 0.001"/>
+      <mesh filename="package://walkie2_description/meshes/CR3base_1.stl" scale="0.001 0.001 0.001"/>
     </geometry>
     <material name="silver"/>
@@ -107,5 +107,5 @@
     <origin xyz="0.016306 -0.0 -0.7855" rpy="0 0 0"/>
     <geometry>
-      <mesh filename="package://walkie2_description/meshes/CR3base_1_1.stl" scale="0.001 0.001 0.001"/>
+      <mesh filename="package://walkie2_description/meshes/CR3base_1.stl" scale="0.001 0.001 0.001"/>
     </geometry>
   </collision>
@@ -120,5 +120,5 @@
     <origin xyz="0.174006 0.05 -1.4942" rpy="0 0 0"/>
     <geometry>
-      <mesh filename="package://walkie2_description/meshes/Realsense_1_1.stl" scale="0.001 0.001 0.001"/>
+      <mesh filename="package://walkie2_description/meshes/Realsense_1.stl" scale="0.001 0.001 0.001"/>
     </geometry>
     <material name="silver"/>
@@ -127,5 +127,5 @@
     <origin xyz="0.174006 0.05 -1.4942" rpy="0 0 0"/>
     <geometry>
-      <mesh filename="package://walkie2_description/meshes/Realsense_1_1.stl" scale="0.001 0.001 0.001"/>
+      <mesh filename="package://walkie2_description/meshes/Realsense_1.stl" scale="0.001 0.001 0.001"/>
     </geometry>
   </collision>

Commit message: fix move group

File: walkie2_ws/src/cr3_lowlevel_pkg/urdf/cr3_robot_w_gripper_for_walkie2.xacro (robot description, xacro)
@@ -285,11 +285,4 @@
     <limit effort="1000" lower="0.0" upper="0.785" velocity="0.2"/>
   </joint>
-    <!-- for Depth Camera -->
-  <xacro:property name="deg_to_rad" value="0.01745329251994329577"/>
-  <xacro:include filename="$(find cr3_lowlevel_pkg)/urdf/_d435.xacro"/>
-  <xacro:sensor_d435 name="sensor_d435" topics_ns="sensor_d435" parent="Link6">
-    <origin xyz="0.031 -0.031 0.0" rpy="1.57 -1.57 0.77"/>
-    <!-- <origin xyz="0 0 0" rpy="${-90.0 * deg_to_rad} 0 ${-90.0 * deg_to_rad}"/> -->
-  </xacro:sensor_d435>
   <!-- xacro implement-->
   <xacro:arm_control transmission="tran_1" joint="joint1" motor="motor_1" />
