Commit message: change xacro to use cr3_robot_w_gripper_for_walkie2, worked

File: walkie2_ws/src/walkie2_description/urdf/walkie2.xacro (robot description, xacro)
@@ -4,23 +4,5 @@
 <xacro:include filename="$(find walkie2_description)/urdf/walkie2.trans" />
 <xacro:include filename="$(find walkie2_description)/urdf/walkie2.gazebo" />
-<xacro:macro name="arm_gazebo" params="link">
-            <gazebo reference="${link}">
-                <material>Gazebo/White</material>
-                <mu1>0.2</mu1>
-                <mu2>0.2</mu2>
-            </gazebo>
-  </xacro:macro>
-  <xacro:macro name="arm_control" params="transmission joint motor">
-    <transmission name="${transmission}">
-      <type>transmission_interface/SimpleTransmission</type>
-      <joint name="${joint}">
-        <hardwareInterface>hardware_interface/PositionJointInterface</hardwareInterface>
-      </joint>
-      <actuator name="${motor}">
-        <hardwareInterface>hardware_interface/PositionJointInterface</hardwareInterface>
-        <mechanicalReduction>1</mechanicalReduction>
-      </actuator>
-    </transmission>
-  </xacro:macro>
+<xacro:include filename="$(find cr3_lowlevel_pkg)/urdf/cr3_robot_w_gripper_for_walkie2.xacro" />
 <link name="base_footprint"/>
 <joint name="base_joint" type="fixed">
@@ -184,293 +166,4 @@
 </joint>
 <link name="imu_link"/>
-<link name="arm_base">
-    <inertial>
-      <origin xyz="0 0 0" rpy="0 0 0" />
-      <mass value="3.06" />
-      <inertia ixx="0.3" ixy="0.0" ixz="0.0" iyy="0.3" iyz="0.0" izz="0.3" />
-    </inertial>
-    <visual>
-      <origin xyz="0 0 0" rpy="0 0 1.57" />
-      <geometry>
-        <mesh filename="package://tesr_ros_cr3_pkg/meshes/base_link.dae" />
-      </geometry>
-    </visual>
-    <collision>
-      <origin xyz="0 0 0" rpy="0 0 0" />
-      <geometry>
-        <mesh filename="package://tesr_ros_cr3_pkg/meshes/base_link.STL" />
-      </geometry>
-    </collision>
-  </link>
-  <joint name="arm_joint" type="fixed">
-    <parent link="base_cr3" />
-    <child link="arm_base" />
-    <origin xyz="0.0 0.0 0.0" rpy="0.0 0.0 0.0" />
-  </joint>
-  <link name="Link1">
-    <inertial>
-      <origin xyz="0 0 0" rpy="0 0 0" />
-      <mass value="3.06" />
-      <inertia ixx="0.3" ixy="0.0" ixz="0.0" iyy="0.3" iyz="0.0" izz="0.3" />
-    </inertial>
-    <visual>
-      <origin xyz="0 0 0" rpy="0 0 -3.14" />
-      <geometry>
-        <mesh filename="package://tesr_ros_cr3_pkg/meshes/Link1.dae" />
-      </geometry>
-    </visual>
-    <collision>
-      <origin xyz="0 0 0" rpy="0 0 0" />
-      <geometry>
-        <mesh filename="package://tesr_ros_cr3_pkg/meshes/Link1.STL" />
-      </geometry>
-    </collision>
-  </link>
-  <joint name="joint1" type="revolute">
-    <origin xyz="0 0 0.1283" rpy="0 0 0" />
-    <parent link="arm_base" />
-    <child link="Link1" />
-    <axis xyz="0 0 1" />
-    <limit lower="-3.14" upper="3.14" effort="1000" velocity="100" />
-    <!-- <dynamics damping="${damping_value}" friction="${friction_value}"/> -->
-  </joint>
-  <link name="Link2">
-    <inertial>
-      <origin xyz="0 0 0" rpy="0 0 0" />
-      <mass value="3.06" />
-      <inertia ixx="0.3" ixy="0.0" ixz="0.0" iyy="0.3" iyz="0.0" izz="0.3" />
-    </inertial>
-    <visual>
-      <origin xyz="0 0 0" rpy="0 3.14 3.14" />
-      <geometry>
-        <mesh filename="package://tesr_ros_cr3_pkg/meshes/Link2.dae" />
-      </geometry>
-    </visual>
-    <collision>
-      <origin xyz="0 0 0" rpy="0 0 0" />
-      <geometry>
-        <mesh filename="package://tesr_ros_cr3_pkg/meshes/Link2.STL" />
-      </geometry>
-    </collision>
-  </link>
-  <joint name="joint2" type="revolute">
-    <origin xyz="0 0 0" rpy="1.5708 1.5708 0" />
-    <parent link="Link1" />
-    <child link="Link2" />
-    <axis xyz="0 0 1" />
-    <limit lower="-3.14" upper="3.14" effort="1000" velocity="100" />
-    <!-- <dynamics damping="${damping_value}" friction="${friction_value}"/> -->
-  </joint>
-  <link name="Link3">
-    <inertial>
-      <origin xyz="0 0 0" rpy="0 0 0" />
-      <mass value="3.06" />
-      <inertia ixx="0.3" ixy="0.0" ixz="0.0" iyy="0.3" iyz="0.0" izz="0.3" />
-    </inertial>
-    <visual>
-      <origin xyz="0 0 0" rpy="3.14 0 0" />
-      <geometry>
-        <mesh filename="package://tesr_ros_cr3_pkg/meshes/Link3.dae" />
-      </geometry>
-    </visual>
-    <collision>
-      <origin xyz="0 0 0" rpy="0 0 0" />
-      <geometry>
-        <mesh filename="package://tesr_ros_cr3_pkg/meshes/Link3.STL" />
-      </geometry>
-    </collision>
-  </link>
-  <joint name="joint3" type="revolute">
-    <origin xyz="-0.274 0 0" rpy="0 0 0" />
-    <parent link="Link2" />
-    <child link="Link3" />
-    <axis xyz="0 0 1" />
-    <limit lower="-2.70" upper="2.70" effort="1000" velocity="100" />
-     <!-- <dynamics damping="${damping_value}" friction="${friction_value}"/> -->
-  </joint>
-  <link name="Link4">
-    <inertial>
-      <origin xyz="0 0 0" rpy="0 0 0" />
-      <mass value="3.06" />
-      <inertia ixx="0.3" ixy="0.0" ixz="0.0" iyy="0.3" iyz="0.0" izz="0.3" />
-    </inertial>
-    <visual>
-      <origin xyz="0 0 0" rpy="0 3.14 3.14" />
-      <geometry>
-        <mesh filename="package://tesr_ros_cr3_pkg/meshes/Link4.dae" />
-      </geometry>
-    </visual>
-    <collision>
-      <origin xyz="0 0 0" rpy="0 0 0" />
-      <geometry>
-        <mesh filename="package://tesr_ros_cr3_pkg/meshes/Link4.STL" />
-      </geometry>
-    </collision>
-  </link>
-  <joint name="joint4" type="revolute">
-    <origin xyz="-0.23 0 0.1283" rpy="0 0 -1.5708" />
-    <parent link="Link3" />
-    <child link="Link4" />
-    <axis xyz="0 0 1" />
-    <limit lower="-3.14" upper="3.14" effort="1000" velocity="100" />
-    <!-- <dynamics damping="${damping_value}" friction="${friction_value}"/> -->
-  </joint>
-  <link name="Link5">
-    <inertial>
-      <origin xyz="0 0 0" rpy="0 0 0" />
-      <mass value="3.06" />
-      <inertia ixx="0.3" ixy="0.0" ixz="0.0" iyy="0.3" iyz="0.0" izz="0.3" />
-    </inertial>
-    <visual>
-      <origin xyz="0 0 0" rpy="0 0 0" />
-      <geometry>
-        <mesh filename="package://tesr_ros_cr3_pkg/meshes/Link5.dae" />
-      </geometry>
-    </visual>
-    <collision>
-      <origin xyz="0 0 0" rpy="0 0 0" />
-      <geometry>
-        <mesh filename="package://tesr_ros_cr3_pkg/meshes/Link5.STL" scale="1.1 1.3 1.3"/>
-      </geometry>
-    </collision>
-  </link>
-  <joint name="joint5" type="revolute">
-    <origin xyz="0 -0.116 0" rpy="1.5708 0 0" />
-    <parent link="Link4" />
-    <child link="Link5" />
-    <axis xyz="0 0 1" />
-    <limit lower="-3.14" upper="3.14" effort="1000" velocity="100" />
-    <!-- <dynamics damping="${damping_value}" friction="${friction_value}"/> -->
-  </joint>
-  <link name="Link6">
-    <inertial>
-      <origin xyz="0 0 0" rpy="0 0 0" />
-      <mass value="3.06" />
-      <inertia ixx="0.3" ixy="0.0" ixz="0.0" iyy="0.3" iyz="0.0" izz="0.3" />
-    </inertial>
-    <visual>
-      <origin xyz="0 0 0" rpy="0 0 0" />
-      <geometry>
-        <mesh filename="package://tesr_ros_cr3_pkg/meshes/Link6.dae" />
-      </geometry>
-    </visual>
-    <collision>
-      <origin xyz="0 0 0" rpy="0 0 0" />
-      <geometry>
-        <mesh filename="package://tesr_ros_cr3_pkg/meshes/Link6.STL" />
-      </geometry>
-    </collision>
-  </link>
-  <joint name="joint6" type="revolute">
-    <origin xyz="0 0.105 0" rpy="-1.5708 0 0" />
-    <parent link="Link5" />d
-    <child link="Link6" />
-    <axis xyz="0 0 1" />
-    <limit lower="-3.14" upper="3.14" effort="1000" velocity="100" />
-    <!-- <dynamics damping="${damping_value}" friction="${friction_value}"/> -->
-  </joint>
-  <link name="hand">
-    <inertial>
-      <origin xyz="0 0 0" rpy="0 0 0" />
-      <mass value="0.6" />
-      <inertia ixx="0.1" ixy="0.0" ixz="0.0" iyy="0.1" iyz="0.0" izz="0.1" />
-    </inertial>
-    <visual>
-      <origin xyz="0.010 0.065 0.05" rpy="1.54 0 0.77" />
-      <geometry>
-        <mesh filename="package://tesr_ros_cr3_pkg/meshes/base_gripper.stl" scale="0.001 0.001 0.001" />
-      </geometry>
-    </visual>
-    <collision>
-      <origin xyz="0.053 0.035 0.05" rpy="1.54 0 0.77" />
-      <geometry>
-        <mesh filename="package://tesr_ros_cr3_pkg/meshes/base_gripper.stl" scale="0.001 0.001 0.001" />
-      </geometry>
-    </collision>
-  </link>
-  <joint name="joint7" type="fixed">
-    <parent link="Link6" />
-    <child link="hand" />
-  </joint>
-  <link name="finger_l">
-    <inertial>
-      <origin xyz="0 0 0" rpy="0 0 0" />
-      <mass value="0.3" />
-      <inertia ixx="0.1" ixy="0.0" ixz="0.0" iyy="0.1" iyz="0.0" izz="0.1" />
-    </inertial>
-    <visual>
-      <origin xyz="0.0 0.05 -0.010" rpy="1.54 0 0.77" />
-      <geometry>
-        <mesh filename="package://tesr_ros_cr3_pkg/meshes/FingerL.stl" scale="0.001 0.001 0.001" />
-      </geometry>
-    </visual>
-    <collision>
-      <origin xyz="0.01 0.05 -0.010" rpy="1.54 0 0.77" />
-      <geometry>
-        <mesh filename="package://tesr_ros_cr3_pkg/meshes/FingerL.stl" scale="0.001 0.001 0.001" />
-      </geometry>
-    </collision>
-  </link>
-  <joint name="joint8" type="revolute">
-    <parent link="hand" />
-    <child link="finger_l" />
-    <origin rpy="0 0 0" xyz="0 0 0.0584"/>
-    <axis xyz="0 1 0"/>
-    <limit effort="1000" lower="-0.785" upper="0.0" velocity="0.2"/>
-  </joint>
-  <link name="finger_r">
-    <inertial>
-      <origin xyz="0 0 0" rpy="0 0 0" />
-      <mass value="0.6" />
-      <inertia ixx="0.1" ixy="0.0" ixz="0.0" iyy="0.1" iyz="0.0" izz="0.1" />
-    </inertial>
-    <visual>
-      <origin xyz="0.0050 0.070 -0.005" rpy="1.54 0 0.77" />
-      <geometry>
-        <mesh filename="package://tesr_ros_cr3_pkg/meshes/FingerR v1.stl" scale="0.001 0.001 0.001" />
-      </geometry>
-    </visual>
-    <collision>
-      <origin xyz="0.0050 0.070 -0.005" rpy="1.54 0 0.77" />
-      <geometry>
-        <mesh filename="package://tesr_ros_cr3_pkg/meshes/FingerR v1.stl" scale="0.001 0.001 0.001" />
-      </geometry>
-    </collision>
-  </link>
-  <joint name="joint9" type="revolute">
-    <parent link="hand" />
-    <child link="finger_r" />
-    <origin rpy="0 0 0" xyz="0 0 0.0584"/>
-    <axis xyz="0 1 0"/>
-    <limit effort="1000" lower="0.0" upper="0.785" velocity="0.2"/>
-  </joint>
-    <!-- for Depth Camera -->
-  <xacro:property name="deg_to_rad" value="0.01745329251994329577"/>
-  <xacro:include filename="$(find tesr_ros_cr3_pkg)/urdf/_d435.xacro"/>
-  <xacro:sensor_d435 name="sensor_d435" topics_ns="sensor_d435" parent="Link6">
-    <origin xyz="0.031 -0.031 0.0" rpy="1.57 -1.57 0.77"/>
-    <!-- <origin xyz="0 0 0" rpy="${-90.0 * deg_to_rad} 0 ${-90.0 * deg_to_rad}"/> -->
-  </xacro:sensor_d435>
-  <!-- xacro implement-->
-  <xacro:arm_control transmission="tran_1" joint="joint1" motor="motor_1" />
-  <xacro:arm_control transmission="tran_2" joint="joint2" motor="motor_2" />
-  <xacro:arm_control transmission="tran_3" joint="joint3" motor="motor_3" />
-  <xacro:arm_control transmission="tran_4" joint="joint4" motor="motor_4" />
-  <xacro:arm_control transmission="tran_5" joint="joint5" motor="motor_5" />
-  <xacro:arm_control transmission="tran_6" joint="joint6" motor="motor_6" />
-  <xacro:arm_control transmission="tran_7" joint="joint8" motor="motor_7" />
-  <xacro:arm_control transmission="tran_8" joint="joint9" motor="motor_8" />
-  <gazebo>
-    <plugin name="gazebo_ros_control" filename="libgazebo_ros_control.so" />
-  </gazebo>
-  <xacro:arm_gazebo link="link0"/>
-        <xacro:arm_gazebo link="link1"/>
-        <xacro:arm_gazebo link="link2"/>
-        <xacro:arm_gazebo link="link3"/>
-        <xacro:arm_gazebo link="link4"/>
-        <xacro:arm_gazebo link="link5"/>
-        <xacro:arm_gazebo link="link6"/>
-        <xacro:arm_gazebo link="hand"/>
-        <xacro:arm_gazebo link="finger_l"/>
-        <xacro:arm_gazebo link="finger_r"/>
+<xacro:cr3_robot parent_link="base_cr3"/>
 </robot>

Commit message: change base link and foot print

File: walkie2_ws/src/walkie2_description/urdf/walkie2.xacro (robot description, xacro)
@@ -12,7 +12,7 @@
 <link name="base_link">
   <inertial>
-    <origin xyz="-0.03921029174333767 -5.934425972055137e-06 0.5802747494402485" rpy="0 0 0"/>
-    <mass value="958.092984136945"/>
-    <inertia ixx="143.304009" iyy="141.886997" izz="24.804848" ixy="-6.5e-05" iyz="0.005171" ixz="13.516138"/>
+    <origin xyz="-0.1608928311021478 -5.96990322223803e-06 0.5834834631581107" rpy="0 0 0"/>
+    <mass value="952.3993400032292"/>
+    <inertia ixx="141.167931" iyy="139.78051" izz="23.866384" ixy="-5.5e-05" iyz="0.005153" ixz="12.651599"/>
   </inertial>
   <visual>
@@ -32,19 +32,19 @@
 <link name="right_wheel">
   <inertial>
-    <origin xyz="-2.222335472355593e-15 0.04902981833717965 0.0" rpy="0 0 0"/>
+    <origin xyz="2.128852395337864e-15 0.03612818166282045 6.938893903907228e-17" rpy="0 0 0"/>
     <mass value="12.73279410998368"/>
-    <inertia ixx="0.02996" iyy="0.051127" izz="0.02996" ixy="-0.0" iyz="0.0" ixz="-0.0"/>
+    <inertia ixx="0.02996" iyy="0.051127" izz="0.02996" ixy="-0.0" iyz="0.0" ixz="0.0"/>
   </inertial>
   <visual>
-    <origin xyz="0.0 0.28 -0.098" rpy="0 0 0"/>
+    <origin xyz="0.0 -0.194 -0.098" rpy="0 0 0"/>
     <geometry>
-      <mesh filename="package://walkie2_description/meshes/LM_1.stl" scale="0.001 0.001 0.001"/>
+      <mesh filename="package://walkie2_description/meshes/RM_1_1.stl" scale="0.001 0.001 0.001"/>
     </geometry>
     <material name="silver"/>
   </visual>
   <collision>
-    <origin xyz="0.0 0.28 -0.098" rpy="0 0 0"/>
+    <origin xyz="0.0 -0.194 -0.098" rpy="0 0 0"/>
     <geometry>
-      <mesh filename="package://walkie2_description/meshes/LM_1.stl" scale="0.001 0.001 0.001"/>
+      <mesh filename="package://walkie2_description/meshes/RM_1_1.stl" scale="0.001 0.001 0.001"/>
     </geometry>
   </collision>
@@ -52,39 +52,19 @@
 <link name="left_wheel">
   <inertial>
-    <origin xyz="2.1545575985072264e-15 -0.049029818337179676 2.7755575615628914e-17" rpy="0 0 0"/>
+    <origin xyz="-2.2204515407301662e-15 -0.049029818337179676 6.938893903907228e-17" rpy="0 0 0"/>
     <mass value="12.73279410998368"/>
-    <inertia ixx="0.02996" iyy="0.051127" izz="0.02996" ixy="-0.0" iyz="-0.0" ixz="0.0"/>
+    <inertia ixx="0.02996" iyy="0.051127" izz="0.02996" ixy="0.0" iyz="0.0" ixz="0.0"/>
   </inertial>
   <visual>
-    <origin xyz="0.0 -0.28 -0.098" rpy="0 0 0"/>
+    <origin xyz="0.0 0.194 -0.098" rpy="0 0 0"/>
     <geometry>
-      <mesh filename="package://walkie2_description/meshes/RM_1.stl" scale="0.001 0.001 0.001"/>
+      <mesh filename="package://walkie2_description/meshes/LM_1_1.stl" scale="0.001 0.001 0.001"/>
     </geometry>
     <material name="silver"/>
   </visual>
   <collision>
-    <origin xyz="0.0 -0.28 -0.098" rpy="0 0 0"/>
+    <origin xyz="0.0 0.194 -0.098" rpy="0 0 0"/>
     <geometry>
-      <mesh filename="package://walkie2_description/meshes/RM_1.stl" scale="0.001 0.001 0.001"/>
-    </geometry>
-  </collision>
-</link>
-<link name="base_cr3">
-  <inertial>
-    <origin xyz="0.1214215 0.0 -0.022599999999999953" rpy="0 0 0"/>
-    <mass value="14.169925233606989"/>
-    <inertia ixx="0.034347" iyy="0.072049" izz="0.101571" ixy="0.0" iyz="0.0" ixz="0.0"/>
-  </inertial>
-  <visual>
-    <origin xyz="-0.103694 -0.0 -0.7855" rpy="0 0 0"/>
-    <geometry>
-      <mesh filename="package://walkie2_description/meshes/CR3base_1.stl" scale="0.001 0.001 0.001"/>
-    </geometry>
-    <material name="silver"/>
-  </visual>
-  <collision>
-    <origin xyz="-0.103694 -0.0 -0.7855" rpy="0 0 0"/>
-    <geometry>
-      <mesh filename="package://walkie2_description/meshes/CR3base_1.stl" scale="0.001 0.001 0.001"/>
+      <mesh filename="package://walkie2_description/meshes/LM_1_1.stl" scale="0.001 0.001 0.001"/>
     </geometry>
   </collision>
@@ -97,14 +77,34 @@
   </inertial>
   <visual>
-    <origin xyz="-0.317 0.0 -0.1955" rpy="0 0 0"/>
+    <origin xyz="-0.197 0.0 -0.1955" rpy="0 0 0"/>
     <geometry>
-      <mesh filename="package://walkie2_description/meshes/lidar_1.stl" scale="0.001 0.001 0.001"/>
+      <mesh filename="package://walkie2_description/meshes/lidar_1_1.stl" scale="0.001 0.001 0.001"/>
     </geometry>
     <material name="silver"/>
   </visual>
   <collision>
-    <origin xyz="-0.317 0.0 -0.1955" rpy="0 0 0"/>
+    <origin xyz="-0.197 0.0 -0.1955" rpy="0 0 0"/>
     <geometry>
-      <mesh filename="package://walkie2_description/meshes/lidar_1.stl" scale="0.001 0.001 0.001"/>
+      <mesh filename="package://walkie2_description/meshes/lidar_1_1.stl" scale="0.001 0.001 0.001"/>
+    </geometry>
+  </collision>
+</link>
+<link name="base_cr3">
+  <inertial>
+    <origin xyz="0.1214215 -1.486984513226704e-17 -0.022599999999999953" rpy="0 0 0"/>
+    <mass value="14.169925233606989"/>
+    <inertia ixx="0.034347" iyy="0.072049" izz="0.101571" ixy="0.0" iyz="0.0" ixz="0.0"/>
+  </inertial>
+  <visual>
+    <origin xyz="0.016306 -0.0 -0.7855" rpy="0 0 0"/>
+    <geometry>
+      <mesh filename="package://walkie2_description/meshes/CR3base_1_1.stl" scale="0.001 0.001 0.001"/>
+    </geometry>
+    <material name="silver"/>
+  </visual>
+  <collision>
+    <origin xyz="0.016306 -0.0 -0.7855" rpy="0 0 0"/>
+    <geometry>
+      <mesh filename="package://walkie2_description/meshes/CR3base_1_1.stl" scale="0.001 0.001 0.001"/>
     </geometry>
   </collision>
@@ -112,24 +112,24 @@
 <link name="realsense">
   <inertial>
-    <origin xyz="-1.3183898417423734e-16 0.050000000000000024 1.3322676295501878e-15" rpy="0 0 0"/>
+    <origin xyz="-1.1102230246251565e-16 0.050000000000000024 1.3322676295501878e-15" rpy="0 0 0"/>
     <mass value="0.3648087412503483"/>
     <inertia ixx="0.000317" iyy="2.7e-05" izz="0.000317" ixy="-0.0" iyz="0.0" ixz="-0.0"/>
   </inertial>
   <visual>
-    <origin xyz="0.054006 0.0 -1.4942" rpy="0 0 0"/>
+    <origin xyz="0.174006 0.05 -1.4942" rpy="0 0 0"/>
     <geometry>
-      <mesh filename="package://walkie2_description/meshes/Realsense_1.stl" scale="0.001 0.001 0.001"/>
+      <mesh filename="package://walkie2_description/meshes/Realsense_1_1.stl" scale="0.001 0.001 0.001"/>
     </geometry>
     <material name="silver"/>
   </visual>
   <collision>
-    <origin xyz="0.054006 0.05 -1.4942" rpy="0 0 0"/>
+    <origin xyz="0.174006 0.05 -1.4942" rpy="0 0 0"/>
     <geometry>
-      <mesh filename="package://walkie2_description/meshes/Realsense_1.stl" scale="0.001 0.001 0.001"/>
+      <mesh filename="package://walkie2_description/meshes/Realsense_1_1.stl" scale="0.001 0.001 0.001"/>
     </geometry>
   </collision>
 </link>
 <joint name="right_wheel_joint" type="continuous">
-  <origin xyz="0.0 -0.28 0.098" rpy="0 0 0"/>
+  <origin xyz="0.0 0.194 0.098" rpy="0 0 0"/>
   <parent link="base_link"/>
   <child link="right_wheel"/>
@@ -137,25 +137,26 @@
 </joint>
 <joint name="left_wheel_joint" type="continuous">
-  <origin xyz="0.0 0.28 0.098" rpy="0 0 0"/>
+  <origin xyz="0.0 -0.194 0.098" rpy="0 0 0"/>
   <parent link="base_link"/>
   <child link="left_wheel"/>
-  <axis xyz="0.0 1.0 0.0"/>
+  <axis xyz="0.0 -1.0 0.0"/>
+</joint>
+<joint name="hokuyo_joint" type="fixed">
+  <origin xyz="0.197 0.0 0.1955" rpy="0 0 0"/>
+  <parent link="base_link"/>
+  <child link="hokuyo"/>
 </joint>
 <joint name="base_cr3_joint" type="prismatic">
-  <origin xyz="0.103694 0.0 0.7855" rpy="0 0 0"/>
+  <origin xyz="-0.016306 0.0 0.7855" rpy="0 0 0"/>
   <parent link="base_link"/>
   <child link="base_cr3"/>
   <axis xyz="0.0 0.0 1.0"/>
-  <limit upper="0.0" lower="-0.3" effort="100" velocity="100"/>
+  <limit upper="0.0" lower="0.0" effort="100" velocity="100"/>
 </joint>
-<joint name="hokuyo_joint" type="fixed">
-  <origin xyz="0.317 0.0 0.1955" rpy="0 0 0"/>
-  <parent link="base_link"/>
-  <child link="hokuyo"/>
-</joint>
-<joint name="realsense_joint" type="fixed">
-  <origin xyz="-0.054006 0 1.4942" rpy="0 0 0"/>
+<joint name="realsense_joint" type="continuous">
+  <origin xyz="-0.174006 -0.05 1.4942" rpy="0 0 0"/>
   <parent link="base_link"/>
   <child link="realsense"/>
+  <axis xyz="0.0 1.0 0.0"/>
 </joint>
 <joint name="imu_joint" type="fixed">

Commit message: update param

File: walkie2_ws/src/walkie2_description/urdf/walkie2.xacro (robot description, xacro)
@@ -155,5 +155,5 @@
   <limit upper="0.0" lower="0.0" effort="100" velocity="100"/>
 </joint>
-<joint name="realsense_joint" type="continuous">
+<joint name="realsense_joint" type="fixed">
   <origin xyz="-0.174006 -0.05 1.4942" rpy="0 0 0"/>
   <parent link="base_link"/>

Commit message: pub joint realsense and lift

File: walkie2_ws/src/walkie2_description/urdf/walkie2.xacro (robot description, xacro)
@@ -155,9 +155,10 @@
   <limit upper="0.0" lower="0.0" effort="100" velocity="100"/>
 </joint>
-<joint name="realsense_joint" type="continuous">
+<joint name="realsense_joint" type="revolute">
   <origin xyz="-0.174006 -0.05 1.4942" rpy="0 0 0"/>
   <parent link="base_link"/>
   <child link="realsense"/>
   <axis xyz="0.0 1.0 0.0"/>
+  <limit effort="1000" lower="0" upper="3.14" velocity="0.2"/>
 </joint>
 <joint name="imu_joint" type="fixed">
