Commit message: add pub joint states urdf realsense pitch yaw

File: walkie2_ws/src/walkie2_description/urdf/walkie2.xacro (robot description, xacro)
@@ -111,5 +111,25 @@
   </collision>
 </link>
-<link name="realsense">
+<link name="realsense_yaw">
+  <inertial>
+    <origin xyz="-0.009267873664598997 -0.009584201347951788 0.0168296234143277" rpy="0 0 0"/>
+    <mass value="0.52273509412428"/>
+    <inertia ixx="0.001265" iyy="0.000145" izz="0.001315" ixy="0.000132" iyz="1.4e-05" ixz="7e-06"/>
+  </inertial>
+  <visual>
+    <origin xyz="0.189306 -0.0 -1.463" rpy="0 0 0"/>
+    <geometry>
+      <mesh filename="package://walkie2_description/meshes/realsense_yaw.stl" scale="0.001 0.001 0.001"/>
+    </geometry>
+    <material name="steel_satin"/>
+  </visual>
+  <collision>
+    <origin xyz="0.189306 -0.0 -1.463" rpy="0 0 0"/>
+    <geometry>
+      <mesh filename="package://walkie2_description/meshes/realsense_yaw.stl" scale="0.001 0.001 0.001"/>
+    </geometry>
+  </collision>
+</link>
+<link name="realsense_pitch">
   <inertial>
     <origin xyz="-1.1102230246251565e-16 0.050000000000000024 1.3322676295501878e-15" rpy="0 0 0"/>
@@ -120,5 +140,5 @@
     <origin xyz="0.174006 0.05 -1.4942" rpy="0 0 0"/>
     <geometry>
-      <mesh filename="package://walkie2_description/meshes/Realsense_1.stl" scale="0.001 0.001 0.001"/>
+      <mesh filename="package://walkie2_description/meshes/realsense_pitch.stl" scale="0.001 0.001 0.001"/>
     </geometry>
     <material name="silver"/>
@@ -127,5 +147,5 @@
     <origin xyz="0.174006 0.05 -1.4942" rpy="0 0 0"/>
     <geometry>
-      <mesh filename="package://walkie2_description/meshes/Realsense_1.stl" scale="0.001 0.001 0.001"/>
+      <mesh filename="package://walkie2_description/meshes/realsense_pitch.stl" scale="0.001 0.001 0.001"/>
     </geometry>
   </collision>
@@ -155,10 +175,17 @@
   <limit upper="0.0" lower="0.0" effort="100" velocity="100"/>
 </joint>
-<joint name="realsense_joint" type="revolute">
-  <origin xyz="-0.174006 -0.05 1.4942" rpy="0 0 0"/>
+<joint name="realsense_yaw_joint" type="revolute">
+  <origin xyz="-0.189306 0.0 1.463" rpy="0 0 0"/>
   <parent link="base_link"/>
-  <child link="realsense"/>
+  <child link="realsense_pitch"/>
+  <axis xyz="0.0 0.0 1.0"/>
+  <limit effort="1000" lower="-1.57" upper="1.57" velocity="0.2"/>
+</joint>
+<joint name="realsense_pitch_joint" type="revolute">
+  <origin xyz="0.0153 -0.00 0.0175" rpy="0 0 0"/>
+  <parent link="realsense_pitch"/>
+  <child link="realsense_yaw"/>
   <axis xyz="0.0 1.0 0.0"/>
-  <limit effort="1000" lower="0" upper="3.14" velocity="0.2"/>
+  <limit effort="1000" lower="-1.57" upper="1.57" velocity="0.2"/>
 </joint>
 <joint name="imu_joint" type="fixed">

Commit message: add realsense yaw and pitch to urdf

File: walkie2_ws/src/walkie2_description/urdf/walkie2.xacro (robot description, xacro)
@@ -139,14 +139,14 @@
   <visual>
     <origin xyz="0.174006 0.05 -1.4942" rpy="0 0 0"/>
-    <geometry>
+    <!-- <geometry>
       <mesh filename="package://walkie2_description/meshes/realsense_pitch.stl" scale="0.001 0.001 0.001"/>
-    </geometry>
+    </geometry> -->
     <material name="silver"/>
   </visual>
   <collision>
     <origin xyz="0.174006 0.05 -1.4942" rpy="0 0 0"/>
-    <geometry>
+    <!-- <geometry>
       <mesh filename="package://walkie2_description/meshes/realsense_pitch.stl" scale="0.001 0.001 0.001"/>
-    </geometry>
+    </geometry> -->
   </collision>
 </link>
@@ -183,5 +183,5 @@
 </joint>
 <joint name="realsense_pitch_joint" type="revolute">
-  <origin xyz="0.0153 -0.00 0.0175" rpy="0 0 0"/>
+  <origin xyz="0.00 0.00 0.0175" rpy="0 0 0"/>
   <parent link="realsense_pitch"/>
   <child link="realsense_yaw"/>

Commit message: swap realsense joint

File: walkie2_ws/src/walkie2_description/urdf/walkie2.xacro (robot description, xacro)
@@ -139,14 +139,14 @@
   <visual>
     <origin xyz="0.174006 0.05 -1.4942" rpy="0 0 0"/>
-    <!-- <geometry>
+    <geometry>
       <mesh filename="package://walkie2_description/meshes/realsense_pitch.stl" scale="0.001 0.001 0.001"/>
-    </geometry> -->
+    </geometry>
     <material name="silver"/>
   </visual>
   <collision>
     <origin xyz="0.174006 0.05 -1.4942" rpy="0 0 0"/>
-    <!-- <geometry>
+    <geometry>
       <mesh filename="package://walkie2_description/meshes/realsense_pitch.stl" scale="0.001 0.001 0.001"/>
-    </geometry> -->
+    </geometry>
   </collision>
 </link>

Commit message: change name realsense pitch and yaw

File: walkie2_ws/src/walkie2_description/urdf/walkie2.xacro (robot description, xacro)
@@ -175,8 +175,8 @@
   <limit upper="0.0" lower="0.0" effort="100" velocity="100"/>
 </joint>
-<joint name="realsense_yaw_joint" type="revolute">
+<joint name="realsense_yaw_join" type="revolute">
   <origin xyz="-0.189306 0.0 1.463" rpy="0 0 0"/>
   <parent link="base_link"/>
-  <child link="realsense_pitch"/>
+  <child link="realsense_yaw"/>
   <axis xyz="0.0 0.0 1.0"/>
   <limit effort="1000" lower="-1.57" upper="1.57" velocity="0.2"/>
@@ -184,6 +184,6 @@
 <joint name="realsense_pitch_joint" type="revolute">
   <origin xyz="0.00 0.00 0.0175" rpy="0 0 0"/>
-  <parent link="realsense_pitch"/>
-  <child link="realsense_yaw"/>
+  <parent link="realsense_yaw"/>
+  <child link="realsense_pitch"/>
   <axis xyz="0.0 1.0 0.0"/>
   <limit effort="1000" lower="-1.57" upper="1.57" velocity="0.2"/>

Commit message: refactor util

File: walkie2_ws/src/walkie2_description/urdf/walkie2.xacro (robot description, xacro)
@@ -175,5 +175,5 @@
   <limit upper="0.0" lower="0.0" effort="100" velocity="100"/>
 </joint>
-<joint name="realsense_yaw_join" type="revolute">
+<joint name="realsense_yaw_joint" type="revolute">
   <origin xyz="-0.189306 0.0 1.463" rpy="0 0 0"/>
   <parent link="base_link"/>

Commit message: hotfix

File: walkie2_ws/src/walkie2_description/urdf/walkie2.xacro (robot description, xacro)
@@ -189,10 +189,12 @@
   <limit effort="1000" lower="-1.57" upper="1.57" velocity="0.2"/>
 </joint>
+<link name="imu_link">
+  <origin xyz="0 0 0" rpy="0 0 180"/>
+</link>
 <joint name="imu_joint" type="fixed">
     <parent link="base_link"/>
     <child link="imu_link"/>
-    <origin xyz="0 0 0" rpy="0 0 0"/>
-</joint>
-<link name="imu_link"/>
+    <origin xyz="0 0 0" rpy="0 0 180"/>
+</joint>
 <xacro:cr3_robot parent_link="base_cr3"/>
 </robot>
